File: OpenAIO-Whoop.kicad_sch (KiCad schematic)
At the start: 40 parts, among them J40 5V, J41 5V, J42 5V, J43 5V, J44 5V, J45 5V, J46 5V, J47 5V, J48 5V, J49 5V, J50 5V, J51 5V, J52 5V, J53 5V, U1 INA186A3IDCKR

Commit message: checkpoint: Bluejay/BLHeli_S part imports + ESC rework notes
EFM8BB51F16G (C6547511), AGM310MAP (C5184858), BY25Q64ESCIG (C50176394)
imported into libs/lib.kicad_sym + lib.pretty + lib.3dshapes.
BLHELI_S_ESC_NOTES.md documents gate-drive research (1S direct drive vs
2S level-shift requirement) and open design decisions.

Co-Authored-By: Claude Fable 5 <noreply@anthropic.com>
Other:
- removed sheet OSD
